Commit message: All the topics of the testing car are working :D

File: src/my_box_bot_description/urdf/box_bot_geometric.urdf (robot description, URDF)
Before this commit: robot box_bot, 11 links, 10 joints
Links:
- removed link body_link
- removed link gyro_link
- removed link lidarB_link
- removed link lidar_link
- removed link struct1_link
- removed link struct2_link
- removed link struct3_link
- removed link wheel1_link
- removed link wheel2_link
- removed link wheel3_link
- removed link wheel4_link
- added link back_pitch_link, mass 0.001; collision sphere radius=0.010; visual sphere radius=0.010
- added link back_roll_link, mass 0.001; collision cylinder length=0.001 radius=0.0045000000000000005; visual cylinder length=0.001 radius=0.0045000000000000005
- added link back_yaw_link, mass 0.001; collision cylinder length=0.001 radius=0.0045000000000000005; visual cylinder length=0.001 radius=0.0045000000000000005
- added link base_link
- added link chassis, mass 0.5; collision box size=0.1 0.1 0.1; visual mesh filename=package://my_box_bot_description/meshes/cute_cube.dae scale=0.1 0.1 0.1
- added link front_pitch_link, mass 0.001; collision sphere radius=0.010; visual sphere radius=0.010
- added link front_roll_link, mass 0.001; collision cylinder length=0.001 radius=0.0045000000000000005; visual cylinder length=0.001 radius=0.0045000000000000005
- added link front_yaw_link, mass 0.001; collision cylinder length=0.001 radius=0.0045000000000000005; visual cylinder length=0.001 radius=0.0045000000000000005
- added link left_wheel, mass 0.05; collision cylinder length=0.001 radius=0.035; visual cylinder length=0.001 radius=0.035
- added link right_wheel, mass 0.05; collision cylinder length=0.001 radius=0.035; visual cylinder length=0.001 radius=0.035
Joints:
- removed joint gyro_joint
- removed joint lidarB_joint
- removed joint lidar_joint
- removed joint struct1_joint
- removed joint struct2_joint
- removed joint struct3_joint
- removed joint wheel1_joint
- removed joint wheel2_joint
- removed joint wheel3_joint
- removed joint wheel4_joint
- added joint back_pitch_joint: type continuous, parent back_roll_link, child back_pitch_link, origin xyz=0 0 0 rpy=0 0 0, axis 0 1 0, limit effort=1000.0 velocity=100.0
- added joint back_roll_joint: type continuous, parent back_yaw_link, child back_roll_link, origin xyz=0 0 0 rpy=0 0 0, axis 1 0 0, limit effort=1000.0 velocity=100.0
- added joint back_yaw_joint: type continuous, parent chassis, child back_yaw_link, origin xyz=-0.04 0 -0.05 rpy=0 0 0, axis 0 0 1, limit effort=1000.0 velocity=100.0
- added joint base_link_joint: type fixed, parent base_link, child chassis, origin xyz=0 0 0 rpy=0 0 0
- added joint front_pitch_joint: type continuous, parent front_roll_link, child front_pitch_link, origin xyz=0 0 0 rpy=0 0 0, axis 0 1 0, limit effort=1000.0 velocity=100.0
- added joint front_roll_joint: type continuous, parent front_yaw_link, child front_roll_link, origin xyz=0 0 0 rpy=0 0 0, axis 1 0 0, limit effort=1000.0 velocity=100.0
- added joint front_yaw_joint: type continuous, parent chassis, child front_yaw_link, origin xyz=0.04 0 -0.05 rpy=0 0 0, axis 0 0 1, limit effort=1000.0 velocity=100.0
- added joint joint_left_wheel: type continuous, parent chassis, child left_wheel, origin xyz=0 0.05 -0.025 rpy=0 0 0, axis 0 1 0, limit effort=10000 velocity=1000
- added joint joint_right_wheel: type continuous, parent chassis, child right_wheel, origin xyz=0 -0.05 -0.025 rpy=0 0 0, axis 0 1 0, limit effort=10000 velocity=1000

File: src/my_box_bot_description/urdf/box_bot_geometric_meshes.urdf (robot description, URDF)
Before this commit: robot box_bot, 11 links, 10 joints
Links:
- removed link body_link
- removed link gyro_link
- removed link lidarB_link
- removed link lidar_link
- removed link struct1_link
- removed link struct2_link
- removed link struct3_link
- removed link wheel1_link
- removed link wheel2_link
- removed link wheel3_link
- removed link wheel4_link
- added link back_pitch_link, mass 0.001; collision sphere radius=0.010; visual sphere radius=0.010
- added link back_roll_link, mass 0.001; collision cylinder length=0.001 radius=0.0045000000000000005; visual cylinder length=0.001 radius=0.0045000000000000005
- added link back_yaw_link, mass 0.001; collision cylinder length=0.001 radius=0.0045000000000000005; visual cylinder length=0.001 radius=0.0045000000000000005
- added link base_link
- added link chassis, mass 0.5; collision box size=0.1 0.1 0.1; visual mesh filename=package://my_box_bot_description/meshes/cute_cube.dae scale=0.1 0.1 0.1
- added link front_pitch_link, mass 0.001; collision sphere radius=0.010; visual sphere radius=0.010
- added link front_roll_link, mass 0.001; collision cylinder length=0.001 radius=0.0045000000000000005; visual cylinder length=0.001 radius=0.0045000000000000005
- added link front_yaw_link, mass 0.001; collision cylinder length=0.001 radius=0.0045000000000000005; visual cylinder length=0.001 radius=0.0045000000000000005
- added link left_wheel, mass 0.05; collision cylinder length=0.001 radius=0.035; visual cylinder length=0.001 radius=0.035
- added link right_wheel, mass 0.05; collision cylinder length=0.001 radius=0.035; visual cylinder length=0.001 radius=0.035
Joints:
- removed joint gyro_joint
- removed joint lidarB_joint
- removed joint lidar_joint
- removed joint struct1_joint
- removed joint struct2_joint
- removed joint struct3_joint
- removed joint wheel1_joint
- removed joint wheel2_joint
- removed joint wheel3_joint
- removed joint wheel4_joint
- added joint back_pitch_joint: type continuous, parent back_roll_link, child back_pitch_link, origin xyz=0 0 0 rpy=0 0 0, axis 0 1 0, limit effort=1000.0 velocity=100.0
- added joint back_roll_joint: type continuous, parent back_yaw_link, child back_roll_link, origin xyz=0 0 0 rpy=0 0 0, axis 1 0 0, limit effort=1000.0 velocity=100.0
- added joint back_yaw_joint: type continuous, parent chassis, child back_yaw_link, origin xyz=-0.04 0 -0.05 rpy=0 0 0, axis 0 0 1, limit effort=1000.0 velocity=100.0
- added joint base_link_joint: type fixed, parent base_link, child chassis, origin xyz=0 0 0 rpy=0 0 0
- added joint front_pitch_joint: type continuous, parent front_roll_link, child front_pitch_link, origin xyz=0 0 0 rpy=0 0 0, axis 0 1 0, limit effort=1000.0 velocity=100.0
- added joint front_roll_joint: type continuous, parent front_yaw_link, child front_roll_link, origin xyz=0 0 0 rpy=0 0 0, axis 1 0 0, limit effort=1000.0 velocity=100.0
- added joint front_yaw_joint: type continuous, parent chassis, child front_yaw_link, origin xyz=0.04 0 -0.05 rpy=0 0 0, axis 0 0 1, limit effort=1000.0 velocity=100.0
- added joint joint_left_wheel: type continuous, parent chassis, child left_wheel, origin xyz=0 0.05 -0.025 rpy=0 0 0, axis 0 1 0, limit effort=10000 velocity=1000
- added joint joint_right_wheel: type continuous, parent chassis, child right_wheel, origin xyz=0 -0.05 -0.025 rpy=0 0 0, axis 0 1 0, limit effort=10000 velocity=1000
