Commit message: Fixing differential wheels

File: src/my_box_bot_description/urdf/box_bot_meshes_collisions_inertias.urdf (robot description, URDF)
Before this commit: robot box_bot, 20 links, 19 joints
Links:
- removed link chassis
- added link base_footprint
- link base_link: mass None -> 0.5; geometry collision box size=0.256 0.150 0.065; visual mesh filename=package://my_box_bot_description/meshes/cute_cube.dae scale=0.256 0.150 0.065
Joints:
- removed joint base_link_joint
- added joint base_footprint_joint: type fixed, parent base_footprint, child base_link, origin xyz=0 0 0.010 rpy=0 0 0
- joint back_yaw_joint: parent chassis -> base_link
- joint front_yaw_joint: parent chassis -> base_link
- joint gyro_joint: parent chassis -> base_link
- joint joint_diff_wheel_L: parent chassis -> base_link
- joint joint_diff_wheel_R: parent chassis -> base_link
- joint joint_left_wheel: parent chassis -> base_link
- joint joint_left_wheel_f: parent chassis -> base_link
- joint joint_right_wheel: parent chassis -> base_link
- joint joint_right_wheel_f: parent chassis -> base_link
- joint struct1_joint: parent chassis -> base_link
- joint struct2_joint: parent chassis -> base_link
- joint struct3_joint: parent chassis -> base_link
